Commit message: Make xacro file readable directly with moveit assistant

File: catapult_description/urdf/ur.urdf.xacro (robot description, xacro)
@@ -1,4 +1,4 @@
 <?xml version="1.0"?>
-<robot xmlns:xacro="http://wiki.ros.org/xacro" name="$(arg name)">
+<robot xmlns:xacro="http://wiki.ros.org/xacro">
   <!-- robot name parameter -->
    <xacro:arg name="name" default="ur"/>

File: catapult_description/urdf/ur_with_gripper.urdf.xacro (robot description, xacro)
@@ -4,7 +4,38 @@
   <xacro:include filename="$(find robotiq_description)/urdf/ur_to_robotiq_adapter.urdf.xacro" />
   <xacro:include filename="$(find robotiq_description)/urdf/robotiq_2f_85_macro.urdf.xacro" />
-  <xacro:ur_to_robotiq prefix="" parent="flange" child="gripper_mount_link"/>
+  <!-- <xacro:ur_to_robotiq prefix="" parent="flange" child="gripper_mount_link"/> -->
+  coupling joint (modified from robotiq_description/ur_to_robotiq_adapter.urdf.xacro)
+  <joint name="ur_to_robotiq_joint" type="fixed">
+    <parent link="flange"/>
+    <child link="ur_to_robotiq_link"/>
+    <origin xyz="0 0 0" rpy="0 ${pi/2} 0"/>
+  </joint>
+  <link name="ur_to_robotiq_link">
+    <visual>
+      <origin xyz="0 0 0" rpy="0 0 0" />
+      <geometry>
+        <mesh filename="package://robotiq_description/meshes/visual/2f_85/ur_to_robotiq_adapter.dae"/>
+      </geometry>
+    </visual>
+    <collision>
+      <origin xyz="0 0 0" rpy="0 0 0"/>
+      <geometry>
+        <mesh filename="package://robotiq_description/meshes/collision/2f_85/ur_to_robotiq_adapter.stl"/>
+      </geometry>
+    </collision>
+    <inertial>
+      <mass value="0.01" />
+      <origin xyz="0 0 0" />
+      <inertia ixx="0.000044" ixy="0.0" ixz="0.0" iyy="0.000027" iyz="0.0" izz="0.000027" />
+    </inertial>
+  </link>
+  <joint name="gripper_side_joint" type="fixed">
+    <parent link="ur_to_robotiq_link"/>
+    <child link="gripper_mount_link"/>
+    <origin xyz="0 0 0.011" rpy="0 0 0"/>
+  </joint>
+  <link name="gripper_mount_link"/>
   <!-- attache gripper -->
-  <xacro:robotiq_gripper name="gripper" prefix="" parent="gripper_mount_link">
+  <xacro:robotiq_gripper name="gripper" prefix="" parent="gripper_mount_link" use_fake_hardware="true">
     <!-- <origin xyz="0 0 0.004" rpy="0 ${-pi/2} ${pi}"/> -->
     <origin xyz="0 0 0.004" rpy="0 0 0"/>
