Commit message: Last changes before giving up

File: catapult_description/urdf/ur.ros2_control.xacro (robot description, xacro)
@@ -125,4 +125,59 @@
         <state_interface name="effort"/>
       </joint>
+      <!-- Joint interfaces -->
+      <!-- With Ignition or Hardware, they handle mimic joints, so we only need this command interface activated -->
+      <joint name="robotiq_85_left_knuckle_joint">
+        <command_interface name="position"/>
+        <state_interface name="position">
+          <param name="initial_value">0.7929</param>
+        </state_interface>
+        <state_interface name="velocity"/>
+      </joint>
+      <joint name="robotiq_85_right_knuckle_joint">
+        <param name="mimic">robotiq_85_left_knuckle_joint</param>
+        <param name="multiplier">-1</param>
+        <command_interface name="position"/>
+        <state_interface name="position"/>
+        <state_interface name="velocity"/>
+      </joint>
+      <joint name="robotiq_85_left_inner_knuckle_joint">
+        <param name="mimic">robotiq_85_left_knuckle_joint</param>
+        <param name="multiplier">1</param>
+        <command_interface name="position"/>
+        <state_interface name="position"/>
+        <state_interface name="velocity"/>
+      </joint>
+      <joint name="robotiq_85_right_inner_knuckle_joint">
+        <param name="mimic">robotiq_85_left_knuckle_joint</param>
+        <param name="multiplier">-1</param>
+        <command_interface name="position"/>
+        <state_interface name="position"/>
+        <state_interface name="velocity"/>
+      </joint>
+      <joint name="robotiq_85_left_finger_tip_joint">
+        <param name="mimic">robotiq_85_left_knuckle_joint</param>
+        <param name="multiplier">-1</param>
+        <command_interface name="position"/>
+        <state_interface name="position"/>
+        <state_interface name="velocity"/>
+      </joint>
+      <joint name="robotiq_85_right_finger_tip_joint">
+        <param name="mimic">robotiq_85_left_knuckle_joint</param>
+        <param name="multiplier">1</param>
+        <command_interface name="position"/>
+        <state_interface name="position"/>
+        <state_interface name="velocity"/>
+      </joint>
+      <gpio name="reactivate_gripper">
+        <command_interface name="reactivate_gripper_cmd"/>
+        <command_interface name="reactivate_gripper_response"/>
+      </gpio>
+      <!-- <joint name="robotiq_85_left_knuckle_joint"> -->
+      <!--   <command_interface name="position"/> -->
+      <!--   <state_interface name="position"> -->
+      <!--     <param name="initial_value">${initial_positions['robotiq_85_left_knuckle_joint']}</param> -->
+      <!--   </state_interface> -->
+      <!--   <state_interface name="velocity"/> -->
+      <!-- </joint> -->
       <xacro:unless value="${sim_gazebo or sim_ignition}">
         <sensor name="${tf_prefix}tcp_fts_sensor">

File: catapult_description/urdf/ur_with_gripper.urdf.xacro (robot description, xacro)
@@ -4,6 +4,6 @@
   <xacro:include filename="$(find robotiq_description)/urdf/ur_to_robotiq_adapter.urdf.xacro" />
   <xacro:include filename="$(find robotiq_description)/urdf/robotiq_2f_85_macro.urdf.xacro" />
-  <!-- <xacro:ur_to_robotiq prefix="" parent="flange" child="gripper_mount_link"/> -->
-  coupling joint (modified from robotiq_description/ur_to_robotiq_adapter.urdf.xacro)
+  <!-- <xacro:ur_to_robotiq prefix="" parent="flange" child="gripper_mount_link"/>
+       coupling joint (modified from robotiq_description/ur_to_robotiq_adapter.urdf.xacro) -->
   <joint name="ur_to_robotiq_joint" type="fixed">
     <parent link="flange"/>
@@ -15,4 +15,5 @@
       <origin xyz="0 0 0" rpy="0 0 0" />
       <geometry>
+        <!-- <mesh filename="file://$(find robotiq_description)/meshes/visual/2f_85/ur_to_robotiq_adapter.dae"/> -->
         <mesh filename="package://robotiq_description/meshes/visual/2f_85/ur_to_robotiq_adapter.dae"/>
       </geometry>
@@ -37,8 +38,23 @@
   <link name="gripper_mount_link"/>
   <!-- attache gripper -->
-  <xacro:robotiq_gripper name="gripper" prefix="" parent="gripper_mount_link" use_fake_hardware="true">
+  <xacro:robotiq_gripper name="gripper" prefix="" parent="gripper_mount_link">
     <!-- <origin xyz="0 0 0.004" rpy="0 ${-pi/2} ${pi}"/> -->
     <origin xyz="0 0 0.004" rpy="0 0 0"/>
   </xacro:robotiq_gripper>
+  <!-- <joint name="robotiq_85_right_knuckle_joint_mimic" type="continuous"> -->
+  <!--   <parent link="robotiq_85_base_link" /> -->
+  <!-- </joint> -->
+  <!-- <joint name="robotiq_85_left_inner_knuckle_joint_mimic" type="continuous"> -->
+  <!--   <parent link="robotiq_85_base_link" /> -->
+  <!-- </joint> -->
+  <!-- <joint name="robotiq_85_right_inner_knuckle_joint_mimic" type="continuous"> -->
+  <!--   <parent link="robotiq_85_base_link" /> -->
+  <!-- </joint> -->
+  <!-- <joint name="robotiq_85_left_finger_tip_joint_mimic" type="continuous"> -->
+  <!--   <parent link="robotiq_85_left_finger_link" /> -->
+  <!-- </joint> -->
+  <!-- <joint name="robotiq_85_right_finger_tip_joint_mimic" type="continuous"> -->
+  <!--   <parent link="robotiq_85_right_finger_link" /> -->
+  <!-- </joint> -->
   <!-- Gazebo grasping plugin -->
   <!-- <gazebo> -->

File: catapult_moveit_config/srdf/ur.srdf.xacro (robot description, xacro)
@@ -5,5 +5,5 @@
   <!-- parameters -->
   <xacro:arg name="prefix" default="" />
-  <xacro:include filename="$(find ur_moveit_config)/srdf/ur_macro.srdf.xacro"/>
+  <xacro:include filename="$(find catapult_moveit_config)/srdf/ur_macro.srdf.xacro"/>
   <xacro:ur_srdf name="$(arg name)" prefix="$(arg prefix)"/>
 </robot>

File: catapult_moveit_config/srdf/ur_macro.srdf.xacro (robot description, xacro)
@@ -12,5 +12,17 @@
     <!--SUBGROUPS - Groups can also be formed by referencing to already defined group names-->
     <group name="${prefix}${name}_manipulator">
-      <chain base_link="${prefix}base_link" tip_link="${prefix}tool0" />
+      <!-- <chain base_link="${prefix}base_link" tip_link="${prefix}tool0" /> -->
+      <chain base_link="${prefix}base_link" tip_link="robotiq_85_left_knuckle_link" />
+    </group>
+    <group name="gripper">
+        <link name="robotiq_85_base_link"/>
+        <link name="robotiq_85_left_inner_knuckle_link"/>
+        <link name="robotiq_85_left_knuckle_link"/>
+        <link name="robotiq_85_left_finger_link"/>
+        <link name="robotiq_85_left_finger_tip_link"/>
+        <link name="robotiq_85_right_inner_knuckle_link"/>
+        <link name="robotiq_85_right_knuckle_link"/>
+        <link name="robotiq_85_right_finger_link"/>
+        <link name="robotiq_85_right_finger_tip_link"/>
     </group>
     <!--GROUP STATES - Purpose - Define a named state for a particular group, in terms of joint values. This is useful to define states like 'folded arms'-->
@@ -39,7 +51,92 @@
       <joint name="${prefix}wrist_3_joint" value="-0.11" />
     </group_state>
-    <!--END EFFECTOR - Purpose - Represent information about an end effector.-->
+    <group_state name="open" group="gripper">
+        <joint name="robotiq_85_left_knuckle_joint" value="0"/>
+    </group_state>
+    <group_state name="close" group="gripper">
+        <joint name="robotiq_85_left_knuckle_joint" value="0.8"/>
+    </group_state>
+    <!--END EFFECTOR: Purpose: Represent information about an end effector.-->
+    <end_effector name="gripper" parent_link="flange" group="gripper" parent_group="ur_manipulator"/>
+    <!--PASSIVE JOINT: Purpose: this element is used to mark joints that are not actuated-->
+    <passive_joint name="robotiq_85_left_inner_knuckle_joint"/>
+    <passive_joint name="robotiq_85_left_finger_tip_joint"/>
+    <passive_joint name="robotiq_85_right_inner_knuckle_joint"/>
+    <passive_joint name="robotiq_85_right_knuckle_joint"/>
+    <passive_joint name="robotiq_85_right_finger_tip_joint"/>
     <!--VIRTUAL JOINT - Purpose - this element defines a virtual joint between a robot link and an external frame of reference (considered fixed with respect to the robot)-->
     <!--DISABLE COLLISIONS - By default it is assumed that any link of the robot could potentially come into collision with any other link in the robot. This tag disables collision checking between a specified pair of links. -->
+    <disable_collisions link1="robotiq_85_base_link" link2="robotiq_85_left_finger_link" reason="Never"/>
+    <disable_collisions link1="robotiq_85_base_link" link2="robotiq_85_left_finger_tip_link" reason="Never"/>
+    <disable_collisions link1="robotiq_85_base_link" link2="robotiq_85_left_inner_knuckle_link" reason="Adjacent"/>
+    <disable_collisions link1="robotiq_85_base_link" link2="robotiq_85_left_knuckle_link" reason="Adjacent"/>
+    <disable_collisions link1="robotiq_85_base_link" link2="robotiq_85_right_finger_link" reason="Never"/>
+    <disable_collisions link1="robotiq_85_base_link" link2="robotiq_85_right_finger_tip_link" reason="Never"/>
+    <disable_collisions link1="robotiq_85_base_link" link2="robotiq_85_right_inner_knuckle_link" reason="Adjacent"/>
+    <disable_collisions link1="robotiq_85_base_link" link2="robotiq_85_right_knuckle_link" reason="Adjacent"/>
+    <disable_collisions link1="robotiq_85_base_link" link2="ur_to_robotiq_link" reason="Adjacent"/>
+    <disable_collisions link1="robotiq_85_base_link" link2="wrist_1_link" reason="Never"/>
+    <disable_collisions link1="robotiq_85_base_link" link2="wrist_2_link" reason="Never"/>
+    <disable_collisions link1="robotiq_85_base_link" link2="wrist_3_link" reason="Never"/>
+    <disable_collisions link1="robotiq_85_left_finger_link" link2="robotiq_85_left_finger_tip_link" reason="Adjacent"/>
+    <disable_collisions link1="robotiq_85_left_finger_link" link2="robotiq_85_left_inner_knuckle_link" reason="Never"/>
+    <disable_collisions link1="robotiq_85_left_finger_link" link2="robotiq_85_left_knuckle_link" reason="Adjacent"/>
+    <disable_collisions link1="robotiq_85_left_finger_link" link2="robotiq_85_right_finger_link" reason="Never"/>
+    <disable_collisions link1="robotiq_85_left_finger_link" link2="robotiq_85_right_finger_tip_link" reason="Never"/>
+    <disable_collisions link1="robotiq_85_left_finger_link" link2="robotiq_85_right_inner_knuckle_link" reason="Never"/>
+    <disable_collisions link1="robotiq_85_left_finger_link" link2="robotiq_85_right_knuckle_link" reason="Never"/>
+    <disable_collisions link1="robotiq_85_left_finger_link" link2="ur_to_robotiq_link" reason="Never"/>
+    <disable_collisions link1="robotiq_85_left_finger_link" link2="wrist_1_link" reason="Never"/>
+    <disable_collisions link1="robotiq_85_left_finger_link" link2="wrist_2_link" reason="Never"/>
+    <disable_collisions link1="robotiq_85_left_finger_link" link2="wrist_3_link" reason="Never"/>
+    <disable_collisions link1="robotiq_85_left_finger_tip_link" link2="robotiq_85_left_inner_knuckle_link" reason="Default"/>
+    <disable_collisions link1="robotiq_85_left_finger_tip_link" link2="robotiq_85_left_knuckle_link" reason="Never"/>
+    <disable_collisions link1="robotiq_85_left_finger_tip_link" link2="robotiq_85_right_finger_link" reason="Never"/>
+    <disable_collisions link1="robotiq_85_left_finger_tip_link" link2="robotiq_85_right_finger_tip_link" reason="Never"/>
+    <disable_collisions link1="robotiq_85_left_finger_tip_link" link2="robotiq_85_right_inner_knuckle_link" reason="Never"/>
+    <disable_collisions link1="robotiq_85_left_finger_tip_link" link2="robotiq_85_right_knuckle_link" reason="Never"/>
+    <disable_collisions link1="robotiq_85_left_finger_tip_link" link2="ur_to_robotiq_link" reason="Never"/>
+    <disable_collisions link1="robotiq_85_left_finger_tip_link" link2="wrist_1_link" reason="Never"/>
+    <disable_collisions link1="robotiq_85_left_finger_tip_link" link2="wrist_2_link" reason="Never"/>
+    <disable_collisions link1="robotiq_85_left_finger_tip_link" link2="wrist_3_link" reason="Never"/>
+    <disable_collisions link1="robotiq_85_left_inner_knuckle_link" link2="robotiq_85_left_knuckle_link" reason="Never"/>
+    <disable_collisions link1="robotiq_85_left_inner_knuckle_link" link2="robotiq_85_right_finger_link" reason="Never"/>
+    <disable_collisions link1="robotiq_85_left_inner_knuckle_link" link2="robotiq_85_right_finger_tip_link" reason="Never"/>
+    <disable_collisions link1="robotiq_85_left_inner_knuckle_link" link2="robotiq_85_right_inner_knuckle_link" reason="Never"/>
+    <disable_collisions link1="robotiq_85_left_inner_knuckle_link" link2="robotiq_85_right_knuckle_link" reason="Never"/>
+    <disable_collisions link1="robotiq_85_left_inner_knuckle_link" link2="ur_to_robotiq_link" reason="Never"/>
+    <disable_collisions link1="robotiq_85_left_inner_knuckle_link" link2="wrist_1_link" reason="Never"/>
+    <disable_collisions link1="robotiq_85_left_inner_knuckle_link" link2="wrist_2_link" reason="Never"/>
+    <disable_collisions link1="robotiq_85_left_inner_knuckle_link" link2="wrist_3_link" reason="Never"/>
+    <disable_collisions link1="robotiq_85_left_knuckle_link" link2="robotiq_85_right_finger_link" reason="Never"/>
+    <disable_collisions link1="robotiq_85_left_knuckle_link" link2="robotiq_85_right_finger_tip_link" reason="Never"/>
+    <disable_collisions link1="robotiq_85_left_knuckle_link" link2="robotiq_85_right_inner_knuckle_link" reason="Never"/>
+    <disable_collisions link1="robotiq_85_left_knuckle_link" link2="robotiq_85_right_knuckle_link" reason="Never"/>
+    <disable_collisions link1="robotiq_85_left_knuckle_link" link2="ur_to_robotiq_link" reason="Never"/>
+    <disable_collisions link1="robotiq_85_left_knuckle_link" link2="wrist_1_link" reason="Never"/>
+    <disable_collisions link1="robotiq_85_left_knuckle_link" link2="wrist_2_link" reason="Never"/>
+    <disable_collisions link1="robotiq_85_left_knuckle_link" link2="wrist_3_link" reason="Never"/>
+    <disable_collisions link1="robotiq_85_right_finger_link" link2="robotiq_85_right_finger_tip_link" reason="Adjacent"/>
+    <disable_collisions link1="robotiq_85_right_finger_link" link2="robotiq_85_right_inner_knuckle_link" reason="Never"/>
+    <disable_collisions link1="robotiq_85_right_finger_link" link2="robotiq_85_right_knuckle_link" reason="Adjacent"/>
+    <disable_collisions link1="robotiq_85_right_finger_link" link2="ur_to_robotiq_link" reason="Never"/>
+    <disable_collisions link1="robotiq_85_right_finger_link" link2="wrist_1_link" reason="Never"/>
+    <disable_collisions link1="robotiq_85_right_finger_link" link2="wrist_2_link" reason="Never"/>
+    <disable_collisions link1="robotiq_85_right_finger_link" link2="wrist_3_link" reason="Never"/>
+    <disable_collisions link1="robotiq_85_right_finger_tip_link" link2="robotiq_85_right_inner_knuckle_link" reason="Default"/>
+    <disable_collisions link1="robotiq_85_right_finger_tip_link" link2="robotiq_85_right_knuckle_link" reason="Never"/>
+    <disable_collisions link1="robotiq_85_right_finger_tip_link" link2="ur_to_robotiq_link" reason="Never"/>
+    <disable_collisions link1="robotiq_85_right_finger_tip_link" link2="wrist_1_link" reason="Never"/>
+    <disable_collisions link1="robotiq_85_right_finger_tip_link" link2="wrist_2_link" reason="Never"/>
+    <disable_collisions link1="robotiq_85_right_finger_tip_link" link2="wrist_3_link" reason="Never"/>
+    <disable_collisions link1="robotiq_85_right_inner_knuckle_link" link2="robotiq_85_right_knuckle_link" reason="Never"/>
+    <disable_collisions link1="robotiq_85_right_inner_knuckle_link" link2="ur_to_robotiq_link" reason="Never"/>
+    <disable_collisions link1="robotiq_85_right_inner_knuckle_link" link2="wrist_1_link" reason="Never"/>
+    <disable_collisions link1="robotiq_85_right_inner_knuckle_link" link2="wrist_2_link" reason="Never"/>
+    <disable_collisions link1="robotiq_85_right_inner_knuckle_link" link2="wrist_3_link" reason="Never"/>
+    <disable_collisions link1="robotiq_85_right_knuckle_link" link2="ur_to_robotiq_link" reason="Never"/>
+    <disable_collisions link1="robotiq_85_right_knuckle_link" link2="wrist_1_link" reason="Never"/>
+    <disable_collisions link1="robotiq_85_right_knuckle_link" link2="wrist_2_link" reason="Never"/>
+    <disable_collisions link1="robotiq_85_right_knuckle_link" link2="wrist_3_link" reason="Never"/>
     <disable_collisions link1="${prefix}base_link" link2="${prefix}base_link_inertia" reason="Adjacent" />
     <disable_collisions link1="${prefix}base_link_inertia" link2="${prefix}shoulder_link" reason="Adjacent" />
