Commit message: Gripper attached with separate controller and move group

File: catapult_description/urdf/ur.ros2_control.xacro (robot description, xacro)
@@ -127,50 +127,50 @@
       <!-- Joint interfaces -->
       <!-- With Ignition or Hardware, they handle mimic joints, so we only need this command interface activated -->
-      <joint name="robotiq_85_left_knuckle_joint">
-        <command_interface name="position"/>
-        <state_interface name="position">
-          <param name="initial_value">0.7929</param>
-        </state_interface>
-        <state_interface name="velocity"/>
-      </joint>
-      <joint name="robotiq_85_right_knuckle_joint">
-        <param name="mimic">robotiq_85_left_knuckle_joint</param>
-        <param name="multiplier">-1</param>
-        <command_interface name="position"/>
-        <state_interface name="position"/>
-        <state_interface name="velocity"/>
-      </joint>
-      <joint name="robotiq_85_left_inner_knuckle_joint">
-        <param name="mimic">robotiq_85_left_knuckle_joint</param>
-        <param name="multiplier">1</param>
-        <command_interface name="position"/>
-        <state_interface name="position"/>
-        <state_interface name="velocity"/>
-      </joint>
-      <joint name="robotiq_85_right_inner_knuckle_joint">
-        <param name="mimic">robotiq_85_left_knuckle_joint</param>
-        <param name="multiplier">-1</param>
-        <command_interface name="position"/>
-        <state_interface name="position"/>
-        <state_interface name="velocity"/>
-      </joint>
-      <joint name="robotiq_85_left_finger_tip_joint">
-        <param name="mimic">robotiq_85_left_knuckle_joint</param>
-        <param name="multiplier">-1</param>
-        <command_interface name="position"/>
-        <state_interface name="position"/>
-        <state_interface name="velocity"/>
-      </joint>
-      <joint name="robotiq_85_right_finger_tip_joint">
-        <param name="mimic">robotiq_85_left_knuckle_joint</param>
-        <param name="multiplier">1</param>
-        <command_interface name="position"/>
-        <state_interface name="position"/>
-        <state_interface name="velocity"/>
-      </joint>
-      <gpio name="reactivate_gripper">
-        <command_interface name="reactivate_gripper_cmd"/>
-        <command_interface name="reactivate_gripper_response"/>
-      </gpio>
+      <!-- <joint name="robotiq_85_left_knuckle_joint"> -->
+      <!--   <command_interface name="position"/> -->
+      <!--   <state_interface name="position"> -->
+      <!--     <param name="initial_value">0.7929</param> -->
+      <!--   </state_interface> -->
+      <!--   <state_interface name="velocity"/> -->
+      <!-- </joint> -->
+      <!-- <joint name="robotiq_85_right_knuckle_joint"> -->
+      <!--   <param name="mimic">robotiq_85_left_knuckle_joint</param> -->
+      <!--   <param name="multiplier">-1</param> -->
+      <!--   <command_interface name="position"/> -->
+      <!--   <state_interface name="position"/> -->
+      <!--   <state_interface name="velocity"/> -->
+      <!-- </joint> -->
+      <!-- <joint name="robotiq_85_left_inner_knuckle_joint"> -->
+      <!--   <param name="mimic">robotiq_85_left_knuckle_joint</param> -->
+      <!--   <param name="multiplier">1</param> -->
+      <!--   <command_interface name="position"/> -->
+      <!--   <state_interface name="position"/> -->
+      <!--   <state_interface name="velocity"/> -->
+      <!-- </joint> -->
+      <!-- <joint name="robotiq_85_right_inner_knuckle_joint"> -->
+      <!--   <param name="mimic">robotiq_85_left_knuckle_joint</param> -->
+      <!--   <param name="multiplier">-1</param> -->
+      <!--   <command_interface name="position"/> -->
+      <!--   <state_interface name="position"/> -->
+      <!--   <state_interface name="velocity"/> -->
+      <!-- </joint> -->
+      <!-- <joint name="robotiq_85_left_finger_tip_joint"> -->
+      <!--   <param name="mimic">robotiq_85_left_knuckle_joint</param> -->
+      <!--   <param name="multiplier">-1</param> -->
+      <!--   <command_interface name="position"/> -->
+      <!--   <state_interface name="position"/> -->
+      <!--   <state_interface name="velocity"/> -->
+      <!-- </joint> -->
+      <!-- <joint name="robotiq_85_right_finger_tip_joint"> -->
+      <!--   <param name="mimic">robotiq_85_left_knuckle_joint</param> -->
+      <!--   <param name="multiplier">1</param> -->
+      <!--   <command_interface name="position"/> -->
+      <!--   <state_interface name="position"/> -->
+      <!--   <state_interface name="velocity"/> -->
+      <!-- </joint> -->
+      <!-- <gpio name="reactivate_gripper"> -->
+      <!--   <command_interface name="reactivate_gripper_cmd"/> -->
+      <!--   <command_interface name="reactivate_gripper_response"/> -->
+      <!-- </gpio> -->
       <!-- <joint name="robotiq_85_left_knuckle_joint"> -->
       <!--   <command_interface name="position"/> -->

File: catapult_description/urdf/ur_with_gripper.urdf.xacro (robot description, xacro)
@@ -4,4 +4,5 @@
   <xacro:include filename="$(find robotiq_description)/urdf/ur_to_robotiq_adapter.urdf.xacro" />
   <xacro:include filename="$(find robotiq_description)/urdf/robotiq_2f_85_macro.urdf.xacro" />
+  <xacro:include filename="$(find catapult_description)/urdf/2f_85.ros2_control.xacro" />
   <!-- <xacro:ur_to_robotiq prefix="" parent="flange" child="gripper_mount_link"/>
        coupling joint (modified from robotiq_description/ur_to_robotiq_adapter.urdf.xacro) -->
@@ -9,5 +10,5 @@
     <parent link="flange"/>
     <child link="ur_to_robotiq_link"/>
-    <origin xyz="0 0 0" rpy="0 ${pi/2} 0"/>
+    <origin xyz="0.004 0 0" rpy="0 ${pi/2} 0"/>
   </joint>
   <link name="ur_to_robotiq_link">
@@ -42,4 +43,6 @@
     <origin xyz="0 0 0.004" rpy="0 0 0"/>
   </xacro:robotiq_gripper>
+  <!-- ros2 control for gripper -->
+  <xacro:robotiq_gripper_ros2_control name="robotiq_gripper_ros2_control" prefix=""/>
   <!-- <joint name="robotiq_85_right_knuckle_joint_mimic" type="continuous"> -->
   <!--   <parent link="robotiq_85_base_link" /> -->

File: catapult_moveit_config/srdf/ur_macro.srdf.xacro (robot description, xacro)
@@ -12,6 +12,6 @@
     <!--SUBGROUPS - Groups can also be formed by referencing to already defined group names-->
     <group name="${prefix}${name}_manipulator">
-      <!-- <chain base_link="${prefix}base_link" tip_link="${prefix}tool0" /> -->
-      <chain base_link="${prefix}base_link" tip_link="robotiq_85_left_knuckle_link" />
+      <chain base_link="${prefix}base_link" tip_link="${prefix}tool0" />
+      <!-- <chain base_link="${prefix}base_link" tip_link="robotiq_85_left_knuckle_link" /> -->
     </group>
     <group name="gripper">
@@ -34,4 +34,5 @@
       <joint name="${prefix}wrist_2_joint" value="0" />
       <joint name="${prefix}wrist_3_joint" value="0" />
+      <!-- <joint name="robotiq_85_left_knuckle_joint" value="0.8"/> -->
     </group_state>
     <group_state name="${prefix}up" group="${prefix}${name}_manipulator">
@@ -42,4 +43,5 @@
       <joint name="${prefix}wrist_2_joint" value="0" />
       <joint name="${prefix}wrist_3_joint" value="0" />
+      <!-- <joint name="robotiq_85_left_knuckle_joint" value="0.8"/> -->
     </group_state>
     <group_state name="${prefix}test_configuration" group="${prefix}${name}_manipulator">
@@ -50,4 +52,5 @@
       <joint name="${prefix}wrist_2_joint" value="-1.6" />
       <joint name="${prefix}wrist_3_joint" value="-0.11" />
+      <!-- <joint name="robotiq_85_left_knuckle_joint" value="0.8"/> -->
     </group_state>
     <group_state name="open" group="gripper">
@@ -55,5 +58,5 @@
     </group_state>
     <group_state name="close" group="gripper">
-        <joint name="robotiq_85_left_knuckle_joint" value="0.8"/>
+        <joint name="robotiq_85_left_knuckle_joint" value="0.7929"/>
     </group_state>
     <!--END EFFECTOR: Purpose: Represent information about an end effector.-->
